File: PCB/HB-SCI-x-MSP.sch (KiCad schematic (older format))
At the start: 27 parts, among them J1 Prog, J2 FTDI, Q1 BC858, SW1 Config, SW2 4x SW, U1 ATmega328P-AU, U2 MSP430F2001IPW, U3 CC1101, Y1 32kHz

Commit message: update PCB
Parts:
- added C6, C7: 12pF, Capacitor_SMD:C_0805_2012Metric_Pad1.15x1.40mm_HandSolder, symbol Device:C_Small
Connections:
- net GND: now also C6.2, C7.2
- net at U2.12 (P2.7/XOUT), Y1.1: now also C7.1
- net at U2.13 (P2.6/XIN/TA1), Y1.2: now also C6.1
Changed lines of the file:
@@
 U 1 1 611641C5
 P 1850 6270
-F 0 "Y1" H 1980 6360 50  0000 C CNN
-F 1 "32kHz" H 1840 6470 50  0000 C CNN
+F 0 "Y1" H 1850 6420 50  0000 C CNN
+F 1 "32kHz" H 1850 6130 50  0000 C CNN
 F 2 "Crystal:Crystal_DS26_D2.0mm_L6.0mm_Horizontal" H 1850 6270 50  0001 C CNN
 F 3 "~" H 1850 6270 50  0001 C CNN
@@
 $EndComp
 Wire Wire Line
-	2000 6270 2140 6270
+	2000 6270 2060 6270
 Wire Wire Line
 	2140 6070 1640 6070
-Wire Wire Line
-	1640 6070 1640 6270
 Wire Wire Line
 	1640 6270 1700 6270
@@
 	1    0    0    -1
 $EndComp
+$Comp
+L Device:C_Small C6
+U 1 1 611E1F7C
+P 1640 6490
+F 0 "C6" H 1500 6560 50  0000 L CNN
+F 1 "12pF" H 1430 6410 50  0000 L CNN
+F 2 "Capacitor_SMD:C_0805_2012Metric_Pad1.15x1.40mm_HandSolder" H 1640 6490 50  0001 C CNN
+F 3 "~" H 1640 6490 50  0001 C CNN
+	1    1640 6490
+	1    0    0    -1
+$EndComp
+$Comp
+L Device:C_Small C7
+U 1 1 611E2B4C
+P 2060 6490
+F 0 "C7" H 2110 6560 50  0000 L CNN
+F 1 "12pF" H 2120 6420 50  0000 L CNN
+F 2 "Capacitor_SMD:C_0805_2012Metric_Pad1.15x1.40mm_HandSolder" H 2060 6490 50  0001 C CNN
+F 3 "~" H 2060 6490 50  0001 C CNN
+	1    2060 6490
+	1    0    0    -1
+$EndComp
+Wire Wire Line
+	1640 6070 1640 6270
+Connection ~ 1640 6270
+Wire Wire Line
+	1640 6270 1640 6390
+Wire Wire Line
+	2060 6390 2060 6270
+Connection ~ 2060 6270
+Wire Wire Line
+	2060 6270 2140 6270
+$Comp
+L power:GND #PWR03
+U 1 1 611E8B89
+P 1640 6590
+F 0 "#PWR03" H 1640 6340 50  0001 C CNN
+F 1 "GND" H 1645 6417 50  0000 C CNN
+F 2 "" H 1640 6590 50  0001 C CNN
+F 3 "" H 1640 6590 50  0001 C CNN
+	1    1640 6590
+	1    0    0    -1
+$EndComp
+$Comp
+L power:GND #PWR04
+U 1 1 611E912C
+P 2060 6590
+F 0 "#PWR04" H 2060 6340 50  0001 C CNN
+F 1 "GND" H 2065 6417 50  0000 C CNN
+F 2 "" H 2060 6590 50  0001 C CNN
+F 3 "" H 2060 6590 50  0001 C CNN
+	1    2060 6590
+	1    0    0    -1
+$EndComp

Commit message: update pcb
Parts:
- added C8: 1n, Capacitor_SMD:C_0805_2012Metric_Pad1.15x1.40mm_HandSolder, symbol Device:C
- added R10: 47k, Resistor_SMD:R_0805_2012Metric_Pad1.15x1.40mm_HandSolder, symbol Device:R
Connections:
- net +BATT: now also R10.2
- net GND: now also C8.2
- net MSP_RST: now also C8.1, R10.1
Other:
- moved on the sheet: C4
Changed lines of the file:
@@
 L Device:C C4
 U 1 1 611A23B6
-P 1280 5800
-F 0 "C4" H 1120 5890 50  0000 L CNN
-F 1 "100n" H 1050 5710 50  0000 L CNN
-F 2 "Capacitor_SMD:C_0805_2012Metric_Pad1.15x1.40mm_HandSolder" H 1318 5650 50  0001 C CNN
-F 3 "~" H 1280 5800 50  0001 C CNN
-	1    1280 5800
+P 990 5950
+F 0 "C4" H 830 6040 50  0000 L CNN
+F 1 "100n" H 760 5860 50  0000 L CNN
+F 2 "Capacitor_SMD:C_0805_2012Metric_Pad1.15x1.40mm_HandSolder" H 1028 5800 50  0001 C CNN
+F 3 "~" H 990 5950 50  0001 C CNN
+	1    990  5950
 	1    0    0    -1
 $EndComp
@@
 L power:+BATT #PWR01
 U 1 1 611A2DDF
-P 1280 5650
-F 0 "#PWR01" H 1280 5500 50  0001 C CNN
-F 1 "+BATT" H 1295 5823 50  0000 C CNN
-F 2 "" H 1280 5650 50  0001 C CNN
-F 3 "" H 1280 5650 50  0001 C CNN
-	1    1280 5650
+P 990 5800
+F 0 "#PWR01" H 990 5650 50  0001 C CNN
+F 1 "+BATT" H 1005 5973 50  0000 C CNN
+F 2 "" H 990 5800 50  0001 C CNN
+F 3 "" H 990 5800 50  0001 C CNN
+	1    990  5800
 	1    0    0    -1
 $EndComp
@@
 L power:GND #PWR02
 U 1 1 611A3816
-P 1280 5950
-F 0 "#PWR02" H 1280 5700 50  0001 C CNN
-F 1 "GND" H 1285 5777 50  0000 C CNN
-F 2 "" H 1280 5950 50  0001 C CNN
-F 3 "" H 1280 5950 50  0001 C CNN
-	1    1280 5950
+P 990 6100
+F 0 "#PWR02" H 990 5850 50  0001 C CNN
+F 1 "GND" H 995 5927 50  0000 C CNN
+F 2 "" H 990 6100 50  0001 C CNN
+F 3 "" H 990 6100 50  0001 C CNN
+	1    990  6100
 	1    0    0    -1
 $EndComp
@@
 Wire Wire Line
 	6410 3770 6590 3770
-Text GLabel 2000 5420 0    50   Input ~ 0
+Text GLabel 2080 4910 0    50   Input ~ 0
 MSP_RST
-Wire Wire Line
-	2000 5420 2140 5420
 Connection ~ 2140 5420
 $Comp
@@
 	1    0    0    -1
 $EndComp
+$Comp
+L power:+BATT #PWR05
+U 1 1 6129576F
+P 1510 5120
+F 0 "#PWR05" H 1510 4970 50  0001 C CNN
+F 1 "+BATT" H 1525 5293 50  0000 C CNN
+F 2 "" H 1510 5120 50  0001 C CNN
+F 3 "" H 1510 5120 50  0001 C CNN
+	1    1510 5120
+	1    0    0    -1
+$EndComp
+$Comp
+L Device:R R10
+U 1 1 61296171
+P 1510 5270
+F 0 "R10" H 1620 5350 50  0000 C CNN
+F 1 "47k" V 1500 5270 50  0000 C CNN
+F 2 "Resistor_SMD:R_0805_2012Metric_Pad1.15x1.40mm_HandSolder" V 1440 5270 50  0001 C CNN
+F 3 "~" H 1510 5270 50  0001 C CNN
+	1    1510 5270
+	-1   0    0    1
+$EndComp
+$Comp
+L Device:C C8
+U 1 1 612969AE
+P 1510 5570
+F 0 "C8" H 1350 5660 50  0000 L CNN
+F 1 "1n" H 1280 5480 50  0000 L CNN
+F 2 "Capacitor_SMD:C_0805_2012Metric_Pad1.15x1.40mm_HandSolder" H 1548 5420 50  0001 C CNN
+F 3 "~" H 1510 5570 50  0001 C CNN
+	1    1510 5570
+	1    0    0    -1
+$EndComp
+$Comp
+L power:GND #PWR06
+U 1 1 61297028
+P 1510 5720
+F 0 "#PWR06" H 1510 5470 50  0001 C CNN
+F 1 "GND" H 1515 5547 50  0000 C CNN
+F 2 "" H 1510 5720 50  0001 C CNN
+F 3 "" H 1510 5720 50  0001 C CNN
+	1    1510 5720
+	1    0    0    -1
+$EndComp
+Wire Wire Line
+	1510 5420 2140 5420
+Connection ~ 1510 5420
+Wire Wire Line
+	2080 4910 2140 4910
+Connection ~ 2140 4910
 $EndSCHEMATC

Commit message: update pcb
Connections:
- net MSP_RST renamed TDIO
- net TEST renamed TCK
Other:
- note added: "Pin-Mapping\n\nMSP AVR\n1.0 === A4 (17)\n1.1 === A3 (16)\n1.2 === A2 (15)\n1.3 === A1 (14)\n\nRST === A5 (18)"
- moved on the sheet: C8, JP1, R10
Changed lines of the file:
@@
 	1640 6270 1700 6270
 Wire Wire Line
-	2140 5420 2140 4910
-Wire Wire Line
-	2140 4910 3500 4910
-Wire Wire Line
-	4210 4910 4210 3220
+	4210 4840 4210 3220
 Wire Wire Line
 	4210 3220 3630 3220
@@
 	6520 4470 6520 4510
 Text GLabel 3940 5420 2    50   Input ~ 0
-TEST
+TCK
 Text GLabel 6410 3870 0    50   Output ~ 0
-TEST
+TCK
 Wire Wire Line
 	6590 3870 6410 3870
 Text GLabel 6410 3770 0    50   Output ~ 0
-MSP_RST
+TDIO
 Wire Wire Line
 	6410 3770 6590 3770
-Text GLabel 2080 4910 0    50   Input ~ 0
-MSP_RST
-Connection ~ 2140 5420
+Text GLabel 1650 5420 0    50   Input ~ 0
+TDIO
 $Comp
 L Jumper:SolderJumper_2_Open JP1
 U 1 1 6113DD72
-P 3650 4910
-F 0 "JP1" H 3650 5115 50  0000 C CNN
-F 1 "Prog/Run" H 3650 5024 50  0000 C CNN
-F 2 "Jumper:SolderJumper-2_P1.3mm_Open_Pad1.0x1.5mm" H 3650 4910 50  0001 C CNN
-F 3 "~" H 3650 4910 50  0001 C CNN
-	1    3650 4910
-	1    0    0    -1
-$EndComp
-Wire Wire Line
-	3800 4910 4210 4910
+P 3650 4840
+F 0 "JP1" H 3650 5045 50  0000 C CNN
+F 1 "Prog/Run" H 3650 4954 50  0000 C CNN
+F 2 "Jumper:SolderJumper-2_P1.3mm_Open_Pad1.0x1.5mm" H 3650 4840 50  0001 C CNN
+F 3 "~" H 3650 4840 50  0001 C CNN
+	1    3650 4840
+	1    0    0    -1
+$EndComp
+Wire Wire Line
+	3800 4840 4210 4840
 $Comp
 L Connector_Generic:Conn_01x06 J2
@@
 L power:+BATT #PWR05
 U 1 1 6129576F
-P 1510 5120
-F 0 "#PWR05" H 1510 4970 50  0001 C CNN
-F 1 "+BATT" H 1525 5293 50  0000 C CNN
-F 2 "" H 1510 5120 50  0001 C CNN
-F 3 "" H 1510 5120 50  0001 C CNN
-	1    1510 5120
+P 2080 5120
+F 0 "#PWR05" H 2080 4970 50  0001 C CNN
+F 1 "+BATT" H 2095 5293 50  0000 C CNN
+F 2 "" H 2080 5120 50  0001 C CNN
+F 3 "" H 2080 5120 50  0001 C CNN
+	1    2080 5120
 	1    0    0    -1
 $EndComp
@@
 L Device:R R10
 U 1 1 61296171
-P 1510 5270
-F 0 "R10" H 1620 5350 50  0000 C CNN
-F 1 "47k" V 1500 5270 50  0000 C CNN
-F 2 "Resistor_SMD:R_0805_2012Metric_Pad1.15x1.40mm_HandSolder" V 1440 5270 50  0001 C CNN
-F 3 "~" H 1510 5270 50  0001 C CNN
-	1    1510 5270
+P 2080 5270
+F 0 "R10" H 2210 5280 50  0000 C CNN
+F 1 "47k" V 2070 5270 50  0000 C CNN
+F 2 "Resistor_SMD:R_0805_2012Metric_Pad1.15x1.40mm_HandSolder" V 2010 5270 50  0001 C CNN
+F 3 "~" H 2080 5270 50  0001 C CNN
+	1    2080 5270
 	-1   0    0    1
 $EndComp
@@
 L Device:C C8
 U 1 1 612969AE
-P 1510 5570
-F 0 "C8" H 1350 5660 50  0000 L CNN
-F 1 "1n" H 1280 5480 50  0000 L CNN
-F 2 "Capacitor_SMD:C_0805_2012Metric_Pad1.15x1.40mm_HandSolder" H 1548 5420 50  0001 C CNN
-F 3 "~" H 1510 5570 50  0001 C CNN
-	1    1510 5570
+P 2080 5570
+F 0 "C8" H 1920 5660 50  0000 L CNN
+F 1 "1n" H 1850 5480 50  0000 L CNN
+F 2 "Capacitor_SMD:C_0805_2012Metric_Pad1.15x1.40mm_HandSolder" H 2118 5420 50  0001 C CNN
+F 3 "~" H 2080 5570 50  0001 C CNN
+	1    2080 5570
 	1    0    0    -1
 $EndComp
@@
 L power:GND #PWR06
 U 1 1 61297028
-P 1510 5720
-F 0 "#PWR06" H 1510 5470 50  0001 C CNN
-F 1 "GND" H 1515 5547 50  0000 C CNN
-F 2 "" H 1510 5720 50  0001 C CNN
-F 3 "" H 1510 5720 50  0001 C CNN
-	1    1510 5720
-	1    0    0    -1
-$EndComp
-Wire Wire Line
-	1510 5420 2140 5420
-Connection ~ 1510 5420
-Wire Wire Line
-	2080 4910 2140 4910
-Connection ~ 2140 4910
+P 2080 5720
+F 0 "#PWR06" H 2080 5470 50  0001 C CNN
+F 1 "GND" H 2085 5547 50  0000 C CNN
+F 2 "" H 2080 5720 50  0001 C CNN
+F 3 "" H 2080 5720 50  0001 C CNN
+	1    2080 5720
+	1    0    0    -1
+$EndComp
+Wire Wire Line
+	2080 5420 2140 5420
+Connection ~ 2080 5420
+Text Notes 4140 7580 0    50   ~ 0
+Pin-Mapping\n\nMSP       AVR\n1.0 === A4 (17)\n1.1 === A3 (16)\n1.2 === A2 (15)\n1.3 === A1 (14)\n\nRST === A5 (18)
+Wire Notes Line
+	4120 7610 4840 7610
+Wire Notes Line
+	4840 7610 4840 6800
+Wire Notes Line
+	4840 6800 4120 6800
+Wire Notes Line
+	4120 6800 4120 7610
+Wire Wire Line
+	2080 5420 1720 5420
+Wire Wire Line
+	1720 5420 1720 4840
+Wire Wire Line
+	1720 4840 3500 4840
+Wire Wire Line
+	1720 5420 1650 5420
+Connection ~ 1720 5420
 $EndSCHEMATC
